Commit message: edit csv

File: urdf/base/base.urdf.xacro (robot description, xacro)
@@ -26,5 +26,5 @@
 	  <inertial>
 		<origin xyz="-0.3 0 0"/>
-		<mass value="45"/>
+		<mass value="25"/>
 		<inertia ixx="1.64890" ixy="0" ixz="-0.21424"
 				 iyy="2.24766" iyz="0"

File: urdf/wheel/wheel.urdf.xacro (robot description, xacro)
@@ -25,5 +25,5 @@
 	  </visual>
 	  <collision>
-		<origin xyz="0 0 0" rpy="${-M_PI/2} 0 0"/>
+		<origin xyz="0 -0.025 0" rpy="${-M_PI/2} 0 0"/>
 		<geometry>
 		  <cylinder radius="${wheel_radius}" length="${wheel_length}"/>
