Commit message: motor parameter setting

File: robots/plat.urdf.xacro (robot description, xacro)
@@ -36,5 +36,5 @@
   <!-- Front LRF -->
   <xacro:lrf_v0 prefix="front" parent="base_link">
-  	<origin xyz="0.045 0 -0.06" rpy="0 ${M_PI} ${M_PI}"/>
+  	<origin xyz="0.045 0 -0.06" rpy="0 0 0"/>
   </xacro:lrf_v0>
   <link name="camera_link"/>

Commit message: apply noetic

File: robots/plat.urdf.xacro (robot description, xacro)
@@ -1,4 +1,4 @@
 <?xml version="1.0"?>
-<robot name="naviton" xmlns:xacro="http://ros.org/wiki/xacro">
+<robot name="plat" xmlns:xacro="http://ros.org/wiki/xacro">
   <xacro:include filename="$(find plat)/urdf/base/base.urdf.xacro"/>
   <xacro:include filename="$(find plat)/urdf/wheel/wheel.urdf.xacro"/>
@@ -10,16 +10,16 @@
   <!-- =============== Link & Joint =============== -->
   <!-- Base -->
-  <link name="base_footprint"/>
-  <xacro:base_v0 parent="base_footprint">
-	<origin xyz="0.07 0 0.2"/>
+  <link name="base_link"/>
+  <xacro:base_v0 parent="base_link">
+	  <origin xyz="0.07 0.0 0.2"/>
   </xacro:base_v0>
   <!-- Wheel -->
   <!-- Right Wheel -->
-  <xacro:wheel_v0 prefix="right" parent="base_link">
+  <xacro:wheel_v0 prefix="right" parent="body_link">
 	  <origin xyz="-0.07 -0.265 -0.102" rpy="0 0 0"/>
 	  <axis xyz="0 1 0"/>
   </xacro:wheel_v0>
   <!-- Left Wheel -->
-  <xacro:wheel_v0 prefix="left" parent="base_link">
+  <xacro:wheel_v0 prefix="left" parent="body_link">
 	  <origin xyz="-0.07 0.265 -0.102" rpy="0 0 ${M_PI}"/>
 	  <axis xyz="0 -1 0"/>
@@ -35,10 +35,10 @@
   </xacro:gim30_v0>-->
   <!-- Front LRF -->
-  <xacro:lrf_v0 prefix="front" parent="base_link">
+  <xacro:lrf_v0 prefix="front" parent="body_link">
   	<origin xyz="0.045 0 -0.06" rpy="0 0 0"/>
   </xacro:lrf_v0>
   <link name="camera_link"/>
   <joint name="lrf_link_joint" type="fixed">
-	  <parent link="base_link"/>
+	  <parent link="body_link"/>
 	  <child link="camera_link"/>
 	  <origin xyz="0 0 0.195"/>
@@ -67,5 +67,5 @@
   <!-- <xacro:wheel_gazebo_control_v0 rate="25"/> -->
   <!--IMU-->
-  <xacro:imu_macro prefix="imu" parent="base_link" xyz="0 0 0"/>
+  <xacro:imu_macro prefix="imu" parent="body_link" xyz="0 0 0"/>
   <!-- LRF -->
   <xacro:lrf_gazebo_v0 topic_name="/urg/scan" prefix="front"
@@ -73,6 +73,6 @@
 					   min_range="0.10" max_range="60.0"/>
   <!-- VHDL-32E -->
-  <HDL-32E parent="base_link" name="velodyne" topic="velodyne_points" hz="10" samples="1024" gpu="true">
+  <xacro:HDL-32E parent="body_link" name="velodyne" topic="velodyne_points" hz="10" samples="1024" gpu="true">
       <origin xyz="-0.12 0 0.79" rpy="0 0 0" />
-  </HDL-32E>
+  </xacro:HDL-32E>
 </robot>

File: urdf/base/base.urdf.xacro (robot description, xacro)
@@ -4,17 +4,16 @@
   <xacro:macro name="base_v0" params="parent *joint_origin">
 	<joint name="base_link_joint" type="fixed">
-	  <insert_block name="joint_origin"/>
+	  <xacro:insert_block name="joint_origin"/>
 	  <parent link="${parent}"/>
-	  <child link="base_link"/>
+	  <child link="body_link"/>
 	</joint>
-	<link name="base_link">
+	<link name="body_link">
 	  <visual>
 	  	<origin xyz="0 0 0.0" rpy="0 0 ${radians(90)}"/>
 		<geometry>
-		 <!--- <mesh filename="package://kcctsim/meshes/DAE/base/base_link.dae"/>-->
 		 	<mesh filename="package://plat/meshes/STL/base/plat_base.stl" scale="0.001 0.001 0.001"/>
 		</geometry>
 		<material name="gray">
-    		<color rgba="0.8 0.8 0.8 2.0"/>
+    		<color rgba="0.8 0.8 0.8 1.0"/>
   		</material>
 	  </visual>

File: urdf/sensors/gim30/gim30.urdf.xacro (robot description, xacro)
@@ -21,5 +21,5 @@
 	  <inertial>
 		<origin xyz="-0.04 0 -0.1"/>
-		<box_inertial mass="0.85" height="0.1" width="0.05" depth="0.25"/>
+		<xacro:box_inertial mass="0.85" height="0.1" width="0.05" depth="0.25"/>
 	  </inertial>
     </link>

File: urdf/sensors/gps/gps.urdf.xacro (robot description, xacro)
@@ -20,5 +20,5 @@
 	  </collision>
 	  <inertial>
-		<cylinder_inertial mass="0.25" radius="0.065" length="0.055"/>
+		<xacro:cylinder_inertial mass="0.25" radius="0.065" length="0.055"/>
 	  </inertial>
 	</link>

File: urdf/sensors/lrf/lrf.urdf.xacro (robot description, xacro)
@@ -5,5 +5,5 @@
   <xacro:macro name="lrf_v0" params="prefix parent *joint_origin">
 	<joint name="${prefix}_lrf_joint" type="fixed">
-	  <insert_block name="joint_origin"/>
+	  <xacro:insert_block name="joint_origin"/>
 	  <parent link="${parent}"/>
 	  <child link="${prefix}_lrf_link"/>
@@ -23,5 +23,5 @@
 	  <inertial>
 		<origin xyz="0 0 -0.0164"/>
-		<box_inertial mass="0.4" height="0.07" width="0.07" depth="0.08"/>
+		<xacro:box_inertial mass="0.4" height="0.07" width="0.07" depth="0.08"/>
 	  </inertial>
 	</link>

File: urdf/wheel/wheel.urdf.xacro (robot description, xacro)
@@ -4,13 +4,13 @@
   <xacro:include filename="$(find plat)/urdf/wheel/wheel.transmission.xacro"/>
   <xacro:include filename="$(find plat)/urdf/wheel/wheel.gazebo.xacro"/>
-  <property name="wheel_radius" value="0.1"/>
-  <property name="wheel_length" value="0.055"/>
-  <property name="wheel_mass" value="1.5"/>
+  <xacro:property name="wheel_radius" value="0.1"/>
+  <xacro:property name="wheel_length" value="0.055"/>
+  <xacro:property name="wheel_mass" value="1.5"/>
   <xacro:macro name="wheel_v0" params="prefix parent *joint_origin *joint_axis">
 	<joint name="${prefix}_wheel_joint" type="continuous">
-	  <insert_block name="joint_origin"/>
+	  <xacro:insert_block name="joint_origin"/>
 	  <parent link="${parent}"/>
 	  <child link="${prefix}_wheel_link"/>
-	  <insert_block name="joint_axis"/>
+	  <xacro:insert_block name="joint_axis"/>
 	</joint>
 	<link name="${prefix}_wheel_link">
@@ -21,5 +21,5 @@
 		</geometry>
 		<material name="black">
-    		<color rgba="0.2 0.2 0.2 2.0"/>
+    		<color rgba="0.2 0.2 0.2 1.0"/>
   		</material>
 	  </visual>
@@ -32,5 +32,5 @@
 	  <inertial>
 		<origin xyz="0 0 0" rpy="${-M_PI/2} 0 0"/>
-		<cylinder_inertial mass="${wheel_mass}"
+		<xacro:cylinder_inertial mass="${wheel_mass}"
 						   radius="${wheel_radius}" length="${wheel_length}"/>
 	  </inertial>

Commit message: run 917 tsukuba

File: robots/plat.urdf.xacro (robot description, xacro)
@@ -36,5 +36,5 @@
   <!-- Front LRF -->
   <xacro:lrf_v0 prefix="front" parent="body_link">
-  	<origin xyz="0.045 0 -0.06" rpy="0 0 0"/>
+  	<origin xyz="-0.045 0 -0.06" rpy="${M_PI} 0 0"/>
   </xacro:lrf_v0>
   <link name="camera_link"/>

Commit message: simulation bug fix

File: robots/plat.urdf.xacro (robot description, xacro)
@@ -73,6 +73,6 @@
 					   min_range="0.10" max_range="60.0"/>
   <!-- VHDL-32E -->
-  <xacro:HDL-32E parent="body_link" name="velodyne" topic="velodyne_points" hz="10" samples="1024" gpu="true">
-      <origin xyz="-0.12 0 0.79" rpy="0 0 0" />
+  <xacro:HDL-32E parent="body_link" name="velodyne" topic="velodyne_points" hz="10" samples="1024" min_angle="-2.14" max_angle="2.14" gpu="true">
+      <origin xyz="-0.12 0 0.79" rpy="0 0 0"/>
   </xacro:HDL-32E>
 </robot>

File: urdf/wheel/wheel.gazebo.xacro (robot description, xacro)
@@ -4,6 +4,6 @@
 	<gazebo reference="${prefix}_wheel_link">
 	  <selfCollide>false</selfCollide>
-      <mu1 value="0.8" />
-      <mu2 value="0.8" />
+      <mu1 value="0.9" />
+      <mu2 value="0.9" />
     </gazebo>
   </xacro:macro>

File: urdf/wheel/wheel.urdf.xacro (robot description, xacro)
@@ -6,5 +6,5 @@
   <xacro:property name="wheel_radius" value="0.1"/>
   <xacro:property name="wheel_length" value="0.055"/>
-  <xacro:property name="wheel_mass" value="1.5"/>
+  <xacro:property name="wheel_mass" value="20.5"/>
   <xacro:macro name="wheel_v0" params="prefix parent *joint_origin *joint_axis">
 	<joint name="${prefix}_wheel_joint" type="continuous">
@@ -17,5 +17,4 @@
 	  <visual>
 		<geometry>
-		  <!--<mesh filename="package://kcctsim/meshes/DAE/wheel/wheel_link.dae"/>-->
 		   <mesh filename="package://plat/meshes/STL/wheel/plat_wheel.stl" scale="0.001 0.001 0.001"/>
 		</geometry>
